File: schematic/_saved_gps_node.sch (KiCad schematic (older format))
At the start: 70 parts, among them IC1 MCP73831/2, J1 Mounting Hole, J10 Test V_RN, J11 AVR ICSP, J12 UART RF, J13 LIPO_BAT, J14 SOLAR, J15 UART GPS, J16 FW_UPDATE, J17 Conn_Coaxial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

Commit message: PCB layout finsihed
Parts:
- removed J10: Test V_RN, Socket_Strips:Socket_Strip_Straight_1x01_Pitch2.54mm, symbol Conn_01x01
Changed lines of the file:
@@
 L GND #PWR034
 U 1 1 5A2CF3F2
-P 1600 5950
-F 0 "#PWR034" H 1600 5700 50  0001 C CNN
-F 1 "GND" V 1600 5750 50  0000 C CNN
-F 2 "" H 1600 5950 50  0001 C CNN
-F 3 "" H 1600 5950 50  0001 C CNN
-	1    1600 5950
+P 1600 5900
+F 0 "#PWR034" H 1600 5650 50  0001 C CNN
+F 1 "GND" V 1600 5700 50  0000 C CNN
+F 2 "" H 1600 5900 50  0001 C CNN
+F 3 "" H 1600 5900 50  0001 C CNN
+	1    1600 5900
 	0    1    1    0
 $EndComp
@@
 	-1   0    0    1
 $EndComp
-$Comp
-L Conn_01x01 J10
-U 1 1 5B5D307F
-P 4350 7500
-F 0 "J10" H 4350 7600 50  0000 C CNN
-F 1 "Test V_RN" H 4350 7400 50  0000 C CNN
-F 2 "Socket_Strips:Socket_Strip_Straight_1x01_Pitch2.54mm" H 4350 7500 50  0001 C CNN
-F 3 "" H 4350 7500 50  0001 C CNN
-	1    4350 7500
-	-1   0    0    1
-$EndComp
 Text Label 4550 7150 0    60   ~ 0
 V_bak
-Text Label 4550 7500 0    60   ~ 0
-V_RN
 NoConn ~ 1650 5800
 NoConn ~ 1650 6100
