File: schematic/v3/Microcontroller.sch (KiCad schematic (older format))
At the start: 38 parts, among them J11 AVR ICSP, J12 UART RF, J15 UART GPS, J6 USB_OTG, SW2 SW_Push, SW3 SW_Push, U4 ATMEGA32U4-AU, Y1 16MHz

Commit message: Cleaned up schematic
Parts:
- C10, C11, C16, C17, C20, C6, C7, C8, C9: footprint Capacitors_SMD:C_0805 -> Capacitor_SMD:C_0805_2012Metric
- C14, C15: footprint (none) -> Capacitor_SMD:C_0805_2012Metric
- D3, D4: footprint LEDs:LED_0805_HandSoldering -> LED_SMD:LED_0805_2012Metric_Pad1.15x1.40mm_HandSolder
- J11: footprint Pin_Headers:Pin_Header_Straight_2x03_Pitch2.54mm -> Connector_PinHeader_2.54mm:PinHeader_2x03_P2.54mm_Vertical
- J12, J15: footprint Pin_Headers:Pin_Header_Straight_1x03_Pitch2.54mm -> Connector_PinHeader_2.54mm:PinHeader_1x03_P2.54mm_Vertical
- R11, R12, R13, R15, R16, R4, R5, R6: footprint Resistors_SMD:R_0805 -> Resistor_SMD:R_0805_2012Metric
- SW2, SW3: footprint Buttons_Switches_SMD:SW_SPST_PTS645 -> Button_Switch_SMD:SW_SPST_PTS645
- U4: footprint Housings_QFP:TQFP-44_10x10mm_Pitch0.8mm -> Package_QFP:TQFP-44_10x10mm_P0.8mm
Changed lines of the file:
@@
 F 0 "J11" H 8900 1900 50  0000 C CNN
 F 1 "AVR ICSP" H 8900 1500 50  0000 C CNN
-F 2 "Pin_Headers:Pin_Header_Straight_2x03_Pitch2.54mm" H 8850 1700 50  0001 C CNN
+F 2 "Connector_PinHeader_2.54mm:PinHeader_2x03_P2.54mm_Vertical" H 8850 1700 50  0001 C CNN
 F 3 "" H 8850 1700 50  0001 C CNN
 	1    8850 1700
@@
 F 0 "J12" H 1900 7100 50  0000 C CNN
 F 1 "UART RF" H 1900 6700 50  0000 C CNN
-F 2 "Pin_Headers:Pin_Header_Straight_1x03_Pitch2.54mm" H 1900 6900 50  0001 C CNN
+F 2 "Connector_PinHeader_2.54mm:PinHeader_1x03_P2.54mm_Vertical" H 1900 6900 50  0001 C CNN
 F 3 "" H 1900 6900 50  0001 C CNN
 	1    1900 6900
@@
 F 0 "J15" H 3200 7100 50  0000 C CNN
 F 1 "UART GPS" H 3200 6700 50  0000 C CNN
-F 2 "Pin_Headers:Pin_Header_Straight_1x03_Pitch2.54mm" H 3200 6900 50  0001 C CNN
+F 2 "Connector_PinHeader_2.54mm:PinHeader_1x03_P2.54mm_Vertical" H 3200 6900 50  0001 C CNN
 F 3 "" H 3200 6900 50  0001 C CNN
 	1    3200 6900
@@
 F 0 "U4" H 4600 5400 50  0000 C CNN
 F 1 "ATMEGA32U4-AU" H 6250 2200 50  0000 C CNN
-F 2 "Housings_QFP:TQFP-44_10x10mm_Pitch0.8mm" H 5550 3700 50  0001 C CIN
+F 2 "Package_QFP:TQFP-44_10x10mm_P0.8mm" H 5550 3700 50  0001 C CIN
 F 3 "" H 6650 4800 50  0001 C CNN
 	1    5550 3700
@@
 F 0 "D4" V 1538 5383 50  0000 R CNN
 F 1 "LED" V 1447 5383 50  0000 R CNN
-F 2 "LEDs:LED_0805_HandSoldering" H 1500 5500 50  0001 C CNN
+F 2 "LED_SMD:LED_0805_2012Metric_Pad1.15x1.40mm_HandSolder" H 1500 5500 50  0001 C CNN
 F 3 "~" H 1500 5500 50  0001 C CNN
 	1    1500 5500
@@
 F 0 "D3" V 1888 5383 50  0000 R CNN
 F 1 "LED" V 1797 5383 50  0000 R CNN
-F 2 "LEDs:LED_0805_HandSoldering" H 1850 5500 50  0001 C CNN
+F 2 "LED_SMD:LED_0805_2012Metric_Pad1.15x1.40mm_HandSolder" H 1850 5500 50  0001 C CNN
 F 3 "~" H 1850 5500 50  0001 C CNN
 	1    1850 5500
@@
 F 0 "R13" H 1570 5196 50  0000 L CNN
 F 1 "1k" H 1570 5105 50  0000 L CNN
-F 2 "Resistors_SMD:R_0805" V 1430 5150 50  0001 C CNN
+F 2 "Resistor_SMD:R_0805_2012Metric" V 1430 5150 50  0001 C CNN
 F 3 "~" H 1500 5150 50  0001 C CNN
 	1    1500 5150
@@
 F 0 "R12" H 1920 5196 50  0000 L CNN
 F 1 "1k" H 1920 5105 50  0000 L CNN
-F 2 "Resistors_SMD:R_0805" V 1780 5150 50  0001 C CNN
+F 2 "Resistor_SMD:R_0805_2012Metric" V 1780 5150 50  0001 C CNN
 F 3 "~" H 1850 5150 50  0001 C CNN
 	1    1850 5150
@@
 F 0 "R16" H 1570 3646 50  0000 L CNN
 F 1 "100k" H 1570 3555 50  0000 L CNN
-F 2 "Resistors_SMD:R_0805" V 1430 3600 50  0001 C CNN
+F 2 "Resistor_SMD:R_0805_2012Metric" V 1430 3600 50  0001 C CNN
 F 3 "~" H 1500 3600 50  0001 C CNN
 	1    1500 3600
@@
 F 0 "C20" H 1186 3554 50  0000 R CNN
 F 1 "100nF" H 1186 3645 50  0000 R CNN
-F 2 "Capacitors_SMD:C_0805" H 1338 3450 50  0001 C CNN
+F 2 "Capacitor_SMD:C_0805_2012Metric" H 1338 3450 50  0001 C CNN
 F 3 "~" H 1300 3600 50  0001 C CNN
 	1    1300 3600
@@
 F 0 "R15" H 1570 3096 50  0000 L CNN
 F 1 "100k" H 1570 3005 50  0000 L CNN
-F 2 "Resistors_SMD:R_0805" V 1430 3050 50  0001 C CNN
+F 2 "Resistor_SMD:R_0805_2012Metric" V 1430 3050 50  0001 C CNN
 F 3 "~" H 1500 3050 50  0001 C CNN
 	1    1500 3050
@@
 F 0 "R4" V 2407 1400 50  0000 C CNN
 F 1 "22" V 2316 1400 50  0000 C CNN
-F 2 "Resistors_SMD:R_0805" V 2130 1400 50  0001 C CNN
+F 2 "Resistor_SMD:R_0805_2012Metric" V 2130 1400 50  0001 C CNN
 F 3 "~" H 2200 1400 50  0001 C CNN
 	1    2200 1400
@@
 F 0 "R5" V 2000 1600 50  0000 C CNN
 F 1 "22" V 2100 1600 50  0000 C CNN
-F 2 "Resistors_SMD:R_0805" V 2130 1600 50  0001 C CNN
+F 2 "Resistor_SMD:R_0805_2012Metric" V 2130 1600 50  0001 C CNN
 F 3 "~" H 2200 1600 50  0001 C CNN
 	1    2200 1600
@@
 F 0 "C17" H 4086 4654 50  0000 R CNN
 F 1 "100nF" H 4086 4745 50  0000 R CNN
-F 2 "Capacitors_SMD:C_0805" H 4238 4550 50  0001 C CNN
+F 2 "Capacitor_SMD:C_0805_2012Metric" H 4238 4550 50  0001 C CNN
 F 3 "~" H 4200 4700 50  0001 C CNN
 	1    4200 4700
@@
 F 0 "C16" H 4085 3854 50  0000 R CNN
 F 1 "1uF" H 4085 3945 50  0000 R CNN
-F 2 "Capacitors_SMD:C_0805" H 4238 3750 50  0001 C CNN
+F 2 "Capacitor_SMD:C_0805_2012Metric" H 4238 3750 50  0001 C CNN
 F 3 "~" H 4200 3900 50  0001 C CNN
 	1    4200 3900
@@
 F 0 "R6" H 10320 1596 50  0000 L CNN
 F 1 "10k" H 10320 1505 50  0000 L CNN
-F 2 "Resistors_SMD:R_0805" V 10180 1550 50  0001 C CNN
+F 2 "Resistor_SMD:R_0805_2012Metric" V 10180 1550 50  0001 C CNN
 F 3 "~" H 10250 1550 50  0001 C CNN
 	1    10250 1550
@@
 F 0 "R11" H 9170 3746 50  0000 L CNN
 F 1 "10k" H 9170 3655 50  0000 L CNN
-F 2 "Resistors_SMD:R_0805" V 9030 3700 50  0001 C CNN
+F 2 "Resistor_SMD:R_0805_2012Metric" V 9030 3700 50  0001 C CNN
 F 3 "~" H 9100 3700 50  0001 C CNN
 	1    9100 3700
@@
 F 0 "SW3" V 9054 4298 50  0000 L CNN
 F 1 "SW_Push" V 9145 4298 50  0000 L CNN
-F 2 "Buttons_Switches_SMD:SW_SPST_PTS645" H 9100 4350 50  0001 C CNN
+F 2 "Button_Switch_SMD:SW_SPST_PTS645" H 9100 4350 50  0001 C CNN
 F 3 "" H 9100 4350 50  0001 C CNN
 	1    9100 4150
@@
 F 0 "SW2" V 10204 2148 50  0000 L CNN
 F 1 "SW_Push" V 10295 2148 50  0000 L CNN
-F 2 "Buttons_Switches_SMD:SW_SPST_PTS645" H 10250 2200 50  0001 C CNN
+F 2 "Button_Switch_SMD:SW_SPST_PTS645" H 10250 2200 50  0001 C CNN
 F 3 "" H 10250 2200 50  0001 C CNN
 	1    10250 2000
@@
 F 0 "C6" H 4650 7000 50  0000 L CNN
 F 1 "4.7uF" H 4650 6700 50  0000 L CNN
-F 2 "Capacitors_SMD:C_0805" H 4638 6700 50  0001 C CNN
+F 2 "Capacitor_SMD:C_0805_2012Metric" H 4638 6700 50  0001 C CNN
 F 3 "~" H 4600 6850 50  0001 C CNN
 	1    4600 6850
@@
 F 0 "C7" H 5150 7000 50  0000 L CNN
 F 1 "100nF" H 5150 6700 50  0000 L CNN
-F 2 "Capacitors_SMD:C_0805" H 5138 6700 50  0001 C CNN
+F 2 "Capacitor_SMD:C_0805_2012Metric" H 5138 6700 50  0001 C CNN
 F 3 "~" H 5100 6850 50  0001 C CNN
 	1    5100 6850
@@
 F 0 "C8" H 5450 7000 50  0000 L CNN
 F 1 "100nF" H 5450 6700 50  0000 L CNN
-F 2 "Capacitors_SMD:C_0805" H 5438 6700 50  0001 C CNN
+F 2 "Capacitor_SMD:C_0805_2012Metric" H 5438 6700 50  0001 C CNN
 F 3 "~" H 5400 6850 50  0001 C CNN
 	1    5400 6850
@@
 F 0 "C9" H 5750 7000 50  0000 L CNN
 F 1 "100nF" H 5750 6700 50  0000 L CNN
-F 2 "Capacitors_SMD:C_0805" H 5738 6700 50  0001 C CNN
+F 2 "Capacitor_SMD:C_0805_2012Metric" H 5738 6700 50  0001 C CNN
 F 3 "~" H 5700 6850 50  0001 C CNN
 	1    5700 6850
@@
 F 0 "C10" H 6050 7000 50  0000 L CNN
 F 1 "100nF" H 6050 6700 50  0000 L CNN
-F 2 "Capacitors_SMD:C_0805" H 6038 6700 50  0001 C CNN
+F 2 "Capacitor_SMD:C_0805_2012Metric" H 6038 6700 50  0001 C CNN
 F 3 "~" H 6000 6850 50  0001 C CNN
 	1    6000 6850
@@
 F 0 "C11" H 6350 7000 50  0000 L CNN
 F 1 "100nF" H 6350 6700 50  0000 L CNN
-F 2 "Capacitors_SMD:C_0805" H 6338 6700 50  0001 C CNN
+F 2 "Capacitor_SMD:C_0805_2012Metric" H 6338 6700 50  0001 C CNN
 F 3 "~" H 6300 6850 50  0001 C CNN
 	1    6300 6850
@@
 F 0 "C14" V 3548 2500 50  0000 C CNN
 F 1 "22pF" V 3639 2500 50  0000 C CNN
-F 2 "" H 3838 2350 50  0001 C CNN
+F 2 "Capacitor_SMD:C_0805_2012Metric" H 3838 2350 50  0001 C CNN
 F 3 "~" H 3800 2500 50  0001 C CNN
 	1    3800 2500
@@
 F 0 "C15" V 3548 2800 50  0000 C CNN
 F 1 "22pF" V 3639 2800 50  0000 C CNN
-F 2 "" H 3838 2650 50  0001 C CNN
+F 2 "Capacitor_SMD:C_0805_2012Metric" H 3838 2650 50  0001 C CNN
 F 3 "~" H 3800 2800 50  0001 C CNN
 	1    3800 2800
