File: schematic/v3/accelerometer.sch (KiCad schematic (older format))
At the start: 3 parts, among them U6 LIS3DH

Commit message: Fixed battery connector, started bom
Parts:
- C26, C27: symbol Device:C -> gps_node-rescue:C-Device
- U6: symbol STM-LISxxx:LIS3DH -> gps_node-rescue:LIS3DH-STM-LISxxx
Changed lines of the file:
@@
 $EndDescr
 $Comp
-L STM-LISxxx:LIS3DH U6
+L gps_node-rescue:LIS3DH-STM-LISxxx U6
 U 1 1 5BEAA49F
 P 6100 3550
@@
 $EndComp
 $Comp
-L Device:C C26
+L gps_node-rescue:C-Device C26
 U 1 1 5BEAA5D1
 P 3800 3550
@@
 $EndComp
 $Comp
-L Device:C C27
+L gps_node-rescue:C-Device C27
 U 1 1 5BEAA6D7
 P 4200 3550

Commit message: Add feedthrough cap for accelerometer
Parts:
- added C?: C_Feedthrough, symbol Device:C_Feedthrough
Connections:
- net labels added: Vcc_accel
- wire segments 32 -> 36
Changed lines of the file:
@@
 L gps_node-rescue:+3V3-power #PWR?
 U 1 1 5BEAA84B
-P 3800 3300
+P 2850 3250
 AR Path="/5BFC4BE8/5BEAA84B" Ref="#PWR?"  Part="1"
 AR Path="/5BEAA84B" Ref="#PWR?"  Part="1"
 AR Path="/5BEAA40F/5BEAA84B" Ref="#PWR0181"  Part="1"
-F 0 "#PWR0181" H 3800 3150 50  0001 C CNN
-F 1 "+3V3" H 3850 3450 50  0000 C CNN
-F 2 "" H 3800 3300 50  0001 C CNN
-F 3 "" H 3800 3300 50  0001 C CNN
-	1    3800 3300
+F 0 "#PWR0181" H 2850 3100 50  0001 C CNN
+F 1 "+3V3" H 2900 3400 50  0000 C CNN
+F 2 "" H 2850 3250 50  0001 C CNN
+F 3 "" H 2850 3250 50  0001 C CNN
+	1    2850 3250
 	1    0    0    -1
 $EndComp
-Wire Wire Line
-	3800 3300 3800 3350
 Wire Wire Line
 	3800 3350 4200 3350
 Wire Wire Line
 	4200 3350 4200 3400
-Connection ~ 3800 3350
 Wire Wire Line
 	3800 3350 3800 3400
 Wire Wire Line
 	4200 3700 4200 3750
-Wire Wire Line
-	4200 3750 3800 3750
-Wire Wire Line
-	3800 3750 3800 3700
 $Comp
 L gps_node-rescue:GND-power #PWR?
 U 1 1 5BEAAC62
-P 3800 3800
+P 3900 3800
 AR Path="/5BFC4BE8/5BEAAC62" Ref="#PWR?"  Part="1"
 AR Path="/5BEAAC62" Ref="#PWR?"  Part="1"
 AR Path="/5BEAA40F/5BEAAC62" Ref="#PWR0182"  Part="1"
-F 0 "#PWR0182" H 3800 3550 50  0001 C CNN
-F 1 "GND" H 3800 3650 50  0000 C CNN
-F 2 "" H 3800 3800 50  0001 C CNN
-F 3 "" H 3800 3800 50  0001 C CNN
-	1    3800 3800
-	1    0    0    -1
-$EndComp
-Wire Wire Line
-	3800 3750 3800 3800
-Connection ~ 3800 3750
-$Comp
-L gps_node-rescue:+3V3-power #PWR?
-U 1 1 5BEAAFA2
-P 6050 2700
-AR Path="/5BFC4BE8/5BEAAFA2" Ref="#PWR?"  Part="1"
-AR Path="/5BEAAFA2" Ref="#PWR?"  Part="1"
-AR Path="/5BEAA40F/5BEAAFA2" Ref="#PWR0183"  Part="1"
-F 0 "#PWR0183" H 6050 2550 50  0001 C CNN
-F 1 "+3V3" H 6100 2850 50  0000 C CNN
-F 2 "" H 6050 2700 50  0001 C CNN
-F 3 "" H 6050 2700 50  0001 C CNN
-	1    6050 2700
+F 0 "#PWR0182" H 3900 3550 50  0001 C CNN
+F 1 "GND" H 3900 3650 50  0000 C CNN
+F 2 "" H 3900 3800 50  0001 C CNN
+F 3 "" H 3900 3800 50  0001 C CNN
+	1    3900 3800
 	1    0    0    -1
 $EndComp
@@
 Wire Wire Line
 	6150 2750 6150 2800
-Connection ~ 6050 2750
-Wire Wire Line
-	6050 2750 6050 2700
 $Comp
 L gps_node-rescue:GND-power #PWR?
@@
 Wire Wire Line
 	6800 3200 6750 3200
+$Comp
+L Device:C_Feedthrough C?
+U 1 1 5BFC9FEB
+P 3400 3450
+F 0 "C?" H 3400 3755 50  0000 C CNN
+F 1 "C_Feedthrough" H 3400 3664 50  0000 C CNN
+F 2 "" V 3400 3450 50  0001 C CNN
+F 3 "~" V 3400 3450 50  0001 C CNN
+	1    3400 3450
+	1    0    0    -1
+$EndComp
+Wire Wire Line
+	3600 3350 3800 3350
+Connection ~ 3800 3350
+Wire Wire Line
+	2850 3250 2850 3350
+Wire Wire Line
+	2850 3350 3200 3350
+Wire Wire Line
+	3400 3550 3400 3750
+Wire Wire Line
+	3400 3750 3800 3750
+Wire Wire Line
+	3800 3700 3800 3750
+Connection ~ 3800 3750
+Wire Wire Line
+	3800 3750 3900 3750
+Wire Wire Line
+	3900 3800 3900 3750
+Connection ~ 3900 3750
+Wire Wire Line
+	3900 3750 4200 3750
+Text Label 4000 3350 0    50   ~ 0
+Vcc_accel
+Text Label 6150 2750 0    50   ~ 0
+Vcc_accel
 $EndSCHEMATC

Commit message: Change accelerometer power label
Connections:
- net Vcc_accel renamed ACCEL_POWER
Changed lines of the file:
@@
 	3900 3750 4200 3750
 Text Label 4000 3350 0    50   ~ 0
-Vcc_accel
+ACCEL_POWER
 Text Label 6150 2750 0    50   ~ 0
-Vcc_accel
+ACCEL_POWER
 $EndSCHEMATC

Commit message: Replace 10uF by 4.7uF and clean up power circuit
Parts:
- C26: value 10uF -> 4.7uF
Changed lines of the file:
@@
 P 3800 3550
 F 0 "C26" H 3915 3596 50  0000 L CNN
-F 1 "10uF" H 3915 3505 50  0000 L CNN
+F 1 "4.7uF" H 3915 3505 50  0000 L CNN
 F 2 "Capacitors_SMD:C_0805" H 3838 3400 50  0001 C CNN
 F 3 "~" H 3800 3550 50  0001 C CNN

Commit message: Cleaned up schematic
Parts:
- C26, C27: footprint Capacitors_SMD:C_0805 -> Capacitor_SMD:C_0805_2012Metric
- C31: renamed from C?; footprint (none) -> gps_node_components:C_FEEDTHROUGH_0805
- U6: footprint lga_16:LGA16-pitch0.5-3mmx3mm -> Package_LGA:LGA-16_3x3mm_P0.5mm_LayoutBorder3x5y
Connections:
- wire segments 36 -> 37
Other:
- moved on the sheet: C26, C27, C31
Changed lines of the file:
@@
 F 0 "U6" H 6500 3050 50  0000 C CNN
 F 1 "LIS3DH" H 6100 3550 50  0000 C CNN
-F 2 "lga_16:LGA16-pitch0.5-3mmx3mm" H 6300 3750 50  0001 C CNN
+F 2 "Package_LGA:LGA-16_3x3mm_P0.5mm_LayoutBorder3x5y" H 6300 3750 50  0001 C CNN
 F 3 "" H 6300 3750 50  0001 C CNN
 	1    6100 3550
@@
 L gps_node-rescue:C-Device C26
 U 1 1 5BEAA5D1
-P 3800 3550
-F 0 "C26" H 3915 3596 50  0000 L CNN
-F 1 "4.7uF" H 3915 3505 50  0000 L CNN
-F 2 "Capacitors_SMD:C_0805" H 3838 3400 50  0001 C CNN
-F 3 "~" H 3800 3550 50  0001 C CNN
-	1    3800 3550
+P 2900 3300
+F 0 "C26" H 3015 3346 50  0000 L CNN
+F 1 "4.7uF" H 3015 3255 50  0000 L CNN
+F 2 "Capacitor_SMD:C_0805_2012Metric" H 2938 3150 50  0001 C CNN
+F 3 "~" H 2900 3300 50  0001 C CNN
+	1    2900 3300
 	1    0    0    -1
 $EndComp
@@
 L gps_node-rescue:C-Device C27
 U 1 1 5BEAA6D7
-P 4200 3550
-F 0 "C27" H 4315 3596 50  0000 L CNN
-F 1 "100nF" H 4315 3505 50  0000 L CNN
-F 2 "Capacitors_SMD:C_0805" H 4238 3400 50  0001 C CNN
-F 3 "~" H 4200 3550 50  0001 C CNN
-	1    4200 3550
+P 3300 3300
+F 0 "C27" H 3415 3346 50  0000 L CNN
+F 1 "100nF" H 3415 3255 50  0000 L CNN
+F 2 "Capacitor_SMD:C_0805_2012Metric" H 3338 3150 50  0001 C CNN
+F 3 "~" H 3300 3300 50  0001 C CNN
+	1    3300 3300
 	1    0    0    -1
 $EndComp
@@
 L gps_node-rescue:+3V3-power #PWR?
 U 1 1 5BEAA84B
-P 2850 3250
+P 1950 3000
 AR Path="/5BFC4BE8/5BEAA84B" Ref="#PWR?"  Part="1"
 AR Path="/5BEAA84B" Ref="#PWR?"  Part="1"
 AR Path="/5BEAA40F/5BEAA84B" Ref="#PWR0181"  Part="1"
-F 0 "#PWR0181" H 2850 3100 50  0001 C CNN
-F 1 "+3V3" H 2900 3400 50  0000 C CNN
-F 2 "" H 2850 3250 50  0001 C CNN
-F 3 "" H 2850 3250 50  0001 C CNN
-	1    2850 3250
-	1    0    0    -1
-$EndComp
-Wire Wire Line
-	3800 3350 4200 3350
-Wire Wire Line
-	4200 3350 4200 3400
-Wire Wire Line
-	3800 3350 3800 3400
-Wire Wire Line
-	4200 3700 4200 3750
+F 0 "#PWR0181" H 1950 2850 50  0001 C CNN
+F 1 "+3V3" H 2000 3150 50  0000 C CNN
+F 2 "" H 1950 3000 50  0001 C CNN
+F 3 "" H 1950 3000 50  0001 C CNN
+	1    1950 3000
+	1    0    0    -1
+$EndComp
+Wire Wire Line
+	2900 3100 3300 3100
+Wire Wire Line
+	3300 3100 3300 3150
+Wire Wire Line
+	2900 3100 2900 3150
+Wire Wire Line
+	3300 3450 3300 3500
 $Comp
 L gps_node-rescue:GND-power #PWR?
 U 1 1 5BEAAC62
-P 3900 3800
+P 3000 3550
 AR Path="/5BFC4BE8/5BEAAC62" Ref="#PWR?"  Part="1"
 AR Path="/5BEAAC62" Ref="#PWR?"  Part="1"
 AR Path="/5BEAA40F/5BEAAC62" Ref="#PWR0182"  Part="1"
-F 0 "#PWR0182" H 3900 3550 50  0001 C CNN
-F 1 "GND" H 3900 3650 50  0000 C CNN
-F 2 "" H 3900 3800 50  0001 C CNN
-F 3 "" H 3900 3800 50  0001 C CNN
-	1    3900 3800
+F 0 "#PWR0182" H 3000 3300 50  0001 C CNN
+F 1 "GND" H 3000 3400 50  0000 C CNN
+F 2 "" H 3000 3550 50  0001 C CNN
+F 3 "" H 3000 3550 50  0001 C CNN
+	1    3000 3550
 	1    0    0    -1
 $EndComp
@@
 	6800 3200 6750 3200
 $Comp
-L Device:C_Feedthrough C?
+L Device:C_Feedthrough C31
 U 1 1 5BFC9FEB
-P 3400 3450
-F 0 "C?" H 3400 3755 50  0000 C CNN
-F 1 "C_Feedthrough" H 3400 3664 50  0000 C CNN
-F 2 "" V 3400 3450 50  0001 C CNN
-F 3 "~" V 3400 3450 50  0001 C CNN
-	1    3400 3450
-	1    0    0    -1
-$EndComp
-Wire Wire Line
-	3600 3350 3800 3350
-Connection ~ 3800 3350
-Wire Wire Line
-	2850 3250 2850 3350
-Wire Wire Line
-	2850 3350 3200 3350
-Wire Wire Line
-	3400 3550 3400 3750
-Wire Wire Line
-	3400 3750 3800 3750
-Wire Wire Line
-	3800 3700 3800 3750
-Connection ~ 3800 3750
-Wire Wire Line
-	3800 3750 3900 3750
-Wire Wire Line
-	3900 3800 3900 3750
-Connection ~ 3900 3750
-Wire Wire Line
-	3900 3750 4200 3750
-Text Label 4000 3350 0    50   ~ 0
+P 2500 3200
+F 0 "C31" H 2500 3505 50  0000 C CNN
+F 1 "C_Feedthrough" H 2500 3414 50  0000 C CNN
+F 2 "gps_node_components:C_FEEDTHROUGH_0805" V 2500 3200 50  0001 C CNN
+F 3 "~" V 2500 3200 50  0001 C CNN
+	1    2500 3200
+	1    0    0    -1
+$EndComp
+Wire Wire Line
+	2700 3100 2900 3100
+Connection ~ 2900 3100
+Wire Wire Line
+	1950 3000 1950 3100
+Wire Wire Line
+	1950 3100 2300 3100
+Wire Wire Line
+	2500 3300 2500 3500
+Wire Wire Line
+	2500 3500 2900 3500
+Wire Wire Line
+	2900 3450 2900 3500
+Connection ~ 2900 3500
+Wire Wire Line
+	2900 3500 3000 3500
+Wire Wire Line
+	3000 3550 3000 3500
+Connection ~ 3000 3500
+Wire Wire Line
+	3000 3500 3300 3500
+Text Label 3100 3100 0    50   ~ 0
 ACCEL_POWER
 Text Label 6150 2750 0    50   ~ 0
 ACCEL_POWER
+Wire Wire Line
+	6150 2750 6500 2750
+Connection ~ 6150 2750
 $EndSCHEMATC
